Commit message: fix + clean-up  description and bringup

File: hk1d_description/ros2_control/hk1d_master_follower.r2c_hardware copy.xacro (robot description, xacro)
@@ -1,8 +1,5 @@
 <?xml version="1.0"?>
 <robot xmlns:xacro="http://www.ros.org/wiki/xacro">
-    <xacro:macro
-        name="kk1d_r2c_hardware"
-        params="prefix use_sim use_fake_hardware command_interface runtime_config_package control_freq">
-    <!-- //////////////////// ROS2 control //////////////////////-->
+    <xacro:macro name="kk1d_r2c_hardware" params="use_fake_hardware command_interface control_freq runtime_config_package">
     <ros2_control name="hk1d_based_system" type="system">
         <xacro:if value="$(arg use_sim)">
@@ -24,11 +21,23 @@
             </hardware>
         </xacro:unless>
-        <xacro:include filename="$(find hk1d_description)/ros2_control/hk1d_macro_import_ec_modules.r2c_hardware.xacro"/>
+        <xacro:include filename="$(find ${hk1d_description})/ros2_control/hk1d_macro_import_ec_modules.r2c_hardware.xacro"/>
+        <!-- master robot -->
         <xacro:hk1d_macro_import_ec_modules
-            prefix="$(arg prefix)"
+            prefix="master_"
             use_fake_hardware="$(arg use_fake_hardware)"
             command_interface="$(arg command_interface)"
-            motor_ec_id="0"
-            sensor_ec_id="1"
+            motor_ec_id=2
+            sensor_ec_id=3
+            ec_config_package="$(find ${runtime_config_package})"
+            ec_motor_config_file="maxon_epos3_config.yaml"
+            ec_sensor_config_file="force_slave_config.yaml"
+        />
+        <!-- follower robot -->
+        <xacro:hk1d_macro_import_ec_modules
+            prefix="follower_"
+            use_fake_hardware="$(arg use_fake_hardware)"
+            command_interface="$(arg command_interface)"
+            motor_ec_id=0
+            sensor_ec_id=1
             ec_config_package="$(find ${runtime_config_package})"
             ec_motor_config_file="maxon_epos3_config.yaml"
